File: light_thing_hw/light_thing_hw.sch (KiCad schematic (older format))
At the start: 23 parts, among them J2 Li-Ion Battery, U1 BC832-V1, U2 LSM6DS3, U3 MCP73832-2-OT, U5A1 STM32L452RETx

Commit message: updates on hw design. it seems like we can make it on a 3x3cm pcb. layout needs work
Parts:
- removed C?: C_Small, symbol Device:C_Small
- removed J?: ST_SWD, symbol Connector_Generic:Conn_01x05
- removed J?: BT_SWD, symbol Connector_Generic:Conn_01x05
- removed L?: INDUCTOR, symbol pspice:INDUCTOR
- removed R?: R, symbol Device:R
- removed RESET_SWITCH1: SW_Push_Dual_x2, Button_Switch_SMD:SW_SPST_B3U-1000P, symbol light_thing_hw-rescue:SW_Push_Dual_x2
- added C10, C8: 10uF, Capacitor_SMD:C_0603_1608Metric_Pad1.05x0.95mm_HandSolder, symbol Device:C_Small
- added C11: 100nF, Capacitor_SMD:C_0603_1608Metric_Pad1.05x0.95mm_HandSolder, symbol Device:C_Small
- added C12: 1nF, Capacitor_SMD:C_0603_1608Metric_Pad1.05x0.95mm_HandSolder, symbol Device:C_Small
- added C13: 100nF, Capacitor_SMD:C_0603_1608Metric_Pad1.05x0.95mm_HandSolder, symbol light_thing_hw-rescue:C_Small
- added D1: 2.5A, Diode_SMD:D_0603_1608Metric_Pad1.05x0.95mm_HandSolder, symbol pspice:DIODE
- added J1: CONNECTORS, Connector_PinHeader_1.00mm:PinHeader_2x04_P1.00mm_Vertical, symbol Connector:Conn_01x08_Female
- added L1: 10uH, 2.5A, Inductor_SMD:L_0603_1608Metric_Pad1.05x0.95mm_HandSolder, symbol Device:L
- added R2: 1M, Resistor_SMD:R_0603_1608Metric_Pad1.05x0.95mm_HandSolder, symbol Device:R
- added R3: 30.1k, Resistor_SMD:R_0603_1608Metric_Pad1.05x0.95mm_HandSolder, symbol Device:R
- added R4: 10k, Resistor_SMD:R_0603_1608Metric_Pad1.05x0.95mm_HandSolder, symbol Device:R
- added R6, R7: R, Resistor_SMD:R_0603_1608Metric_Pad1.05x0.95mm_HandSolder, symbol Device:R
- added SW1: ST_USER_BUTTON1, Button_Switch_THT:SW_Tactile_SPST_Angled_PTS645Vx39-2LFS, symbol Switch:SW_Push
- added SW2: ST_RESET_BUTTON, Button_Switch_SMD:SW_SPST_CK_RS282G05A3, symbol Switch:SW_Push
- C5: value C_Small -> 4.7uF
- C7: renamed from C?; footprint (none) -> Capacitor_SMD:C_0603_1608Metric_Pad1.05x0.95mm_HandSolder
- gave numbers to parts that had none: 1
Connections:
- net labels added: +5V, ACCEL_EXTI_1, ACCEL_EXTI_2, BUTTON1
- wire segments 96 -> 126
Other:
- note added: "BLE AND ACCEL"
- note added: "POWER"
- note added: "UART4 RX"
- note added: "UART4 TX"
- moved on the sheet: C1, C2, C3, C4, C5, C6, C7, J2, R1, U1, U2, U4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

Commit message: hw updates
Parts:
- removed D1: 2.5A, Diode_SMD:D_0603_1608Metric_Pad1.05x0.95mm_HandSolder, symbol pspice:DIODE
- removed J1: CONNECTORS, Connector_PinHeader_1.00mm:PinHeader_2x04_P1.00mm_Vertical, symbol Connector:Conn_01x08_Female
- removed U3: MCP73832-2-OT, Package_TO_SOT_SMD:SOT-23-5, symbol Battery_Management:MCP73832-2-OT
- added 1k1: R, Resistor_SMD:R_0603_1608Metric_Pad1.05x0.95mm_HandSolder, symbol Device:R
- added C14: 10uF, Capacitor_SMD:C_0603_1608Metric_Pad1.05x0.95mm_HandSolder, symbol Device:C_Small
- added C16, C17: 0.1uF, Capacitor_SMD:C_0603_1608Metric_Pad1.05x0.95mm_HandSolder, symbol light_thing_hw-rescue:C_Small
- added D1: 2.5A, 20V, Diode_SMD:D_SOD-323_HandSoldering, symbol Device:D_Schottky_Small
- added D2: GREEN LED, LED_SMD:LED_1806_4516Metric_Pad1.57x1.80mm_HandSolder, symbol Device:LED
- added D3: RED LED, LED_SMD:LED_1806_4516Metric_Pad1.57x1.80mm_HandSolder, symbol Device:LED
- added J1: CONNECTORS, Connector_PinHeader_1.00mm:PinHeader_2x05_P1.00mm_Vertical, symbol Connector:Conn_01x10_Female
- added J3: ADDR_LED_PANEL_1_CONNECTORS, Connector_PinHeader_1.00mm:PinHeader_2x02_P1.00mm_Vertical, symbol Connector:Conn_01x04_Female
- added J4: ADDR_LED_PANEL_2_CONNECTORS, Connector_PinHeader_1.00mm:PinHeader_2x02_P1.00mm_Vertical, symbol Connector:Conn_01x04_Female
- added Q1: MMBF170, Package_TO_SOT_SMD:SOT-23, symbol Transistor_FET:MMBF170
- added R10, R11, R12, R13: 4.7k, Resistor_SMD:R_0603_1608Metric_Pad1.05x0.95mm_HandSolder, symbol Device:R
- added R14: 1k, Resistor_SMD:R_0603_1608Metric_Pad1.05x0.95mm_HandSolder, symbol Device:R
- added R15, R16: 3.5k, Resistor_SMD:R_0603_1608Metric_Pad1.05x0.95mm_HandSolder, symbol Device:R
- added R8, R9: 510, Resistor_SMD:R_0603_1608Metric_Pad1.05x0.95mm_HandSolder, symbol Device:R
- added U3: MCP73833T-FCI_MF, footprints:MCP73833T-FCI&slash_MF, symbol 2020-06-09_04-46-27:MCP73833T-FCI_MF
- added U5: LP38511MRX-ADJ_NOPB, footprints:LP38511MRX-ADJ_NOPB, symbol 2020-06-13_06-34-29:LP38511MRX-ADJ_NOPB
- C1, C2, C3, C4: value 100 nF -> 0.1uF
- C5, C6: value 4.7uF -> 1uF
- R1: value 2k -> 800
- U1: footprint Fanstel_modules:BC832-BC832 -> Fanstel_modules:BC832-BC832_3d1
Connections:
- net labels added: BATT_ADC, BATT_ADC_ENABLE, BT_GPIO_0, BT_GPIO_1, BT_GPIO_2, BT_GPIO_3, BT_RED_LED, GREEN_LED
- net labels removed: BOOT0, USB_ID
- wire segments 126 -> 200
- no-connect marks 1 -> 55
Other:
- note added: "1200mA max current output\n(for 1000mA, have PROG be 1k)"
- note added: "BATTERY: \n- 1100mAH, 40.5mm x 41.5mm x 6.1mm, li-po battery. (3.0V - 4.2V)\nhttps://www.digikey.com/product-detail/en/tinycircuits/ASR00008/1832-1044-ND/8680974"
- moved on the sheet: C10, C12, C7, C8, J2, L1, R2, R3, R4, U1, U4, USB_MICRO_CONN1

Commit message: hw updates
Parts:
- removed R2: 1M, Resistor_SMD:R_0603_1608Metric_Pad1.05x0.95mm_HandSolder, symbol Device:R
- removed U3: MCP73833T-FCI_MF, footprints:MCP73833T-FCI&slash_MF, symbol 2020-06-09_04-46-27:MCP73833T-FCI_MF
- added R17: 1k, Resistor_SMD:R_0603_1608Metric_Pad1.05x0.95mm_HandSolder, symbol Device:R
- added U3: MCP73833T-FCI_UN, footprints:MCP73833T-FCIUN-SMD, symbol MCP73833T-FCI_UN:MCP73833T-FCI_UN
- R1: value 800 -> 470
- R2: renamed from 1k1; value R -> 1k
Connections:
- net +5V: now also R17.1, U3.5 (VSS); no longer C6.2, R1.1
- net VBUS: now also R1.1, U3.1 (VDD_2), U3.2 (VDD)
- net BOOST_ENABLE: now reaches U5A1.38 (PC7)
- net BOOST_ENABLE: now also U4.4 (EN)
- net at R1.2: now also U3.7 (*PG)
- new net: C6.2, U3.10 (VBAT), U3.9 (VBAT_2)
- new net: R17.2, U3.6 (PROG)
- no-connect marks 55 -> 54
Other:
- note removed: "1200mA max current output\n(for 1000mA, have PROG be 1k)"

Commit message: made 5cm pcb. need to do routing etc.
Parts:
- added C15: 2700pF, Capacitor_SMD:C_0603_1608Metric_Pad1.05x0.95mm_HandSolder, symbol Device:C_Small
- added C18: 10uF, Capacitor_SMD:C_0603_1608Metric_Pad1.05x0.95mm_HandSolder, symbol Device:C_Small
- D2, D3: footprint LED_SMD:LED_1806_4516Metric_Pad1.57x1.80mm_HandSolder -> LED_SMD:LED_0603_1608Metric_Pad1.05x0.95mm_HandSolder
- R1: value 470 -> 1k
- R15: value 3.5k -> 2k
- R16: value 3.5k -> 357
- R6: value R -> 4.7k
- R7: value R -> 100
- SW1: footprint Button_Switch_THT:SW_Tactile_SPST_Angled_PTS645Vx39-2LFS -> Button_Switch_SMD:SW_SPST_B3U-3000P
Connections:
- net +3V3: now also C15.2, C18.2
- net +5V: no longer C1.2, C10.2, C11.2, C14.2, C16.2, C17.2, C2.2, C3.2, C4.2, C5.2, C7.2, C8.1, C9.2, D2.1 (K), D3.1 (K), J2.1 (Pin_1), J3.1 (Pin_1), J3.4 (Pin_4), J4.1 (Pin_1), J4.4 (Pin_4), Q1.2 (S), R16.1, R17.1, R4.2, R5.2, R6.2, R7.1, SW1.1, SW2.1, U1.P$1 (GND), U2.1 (SDO/SA0), U2.2 (SDX), U2.3 (SCX), U2.6 (GND), U2.7 (GND), U3.5 (VSS), U4.2 (GND), U5.5 (GND), U5.9 (HEAT_TAB), U5A1.12 (VSSA), U5A1.18 (VSS), U5A1.31 (VSS), U5A1.47 (VSS), U5A1.63 (VSS), USB_MICRO_CONN1.5 (GND)
- net I2C2_SDA: now also U5A1.30 (PB11); no longer U5A1.35 (PB14)
- net CHARGER_STAT2: now reaches U5A1.36 (PB15)
- net CHARGER_STAT2: now also U3.4 (STAT2)
- net GND: now reaches USB_MICRO_CONN1.6 (Shield)
- net GND: now also C1.2, C10.2, C11.2, C14.2, C16.2, C17.2, C2.2, C3.2, C4.2, C5.2, C7.2, C8.1, C9.2, D2.1 (K), D3.1 (K), J2.1 (Pin_1), J3.1 (Pin_1), J3.4 (Pin_4), J4.1 (Pin_1), J4.4 (Pin_4), Q1.2 (S), R16.1, R17.1, R4.2, R5.2, R6.2, R7.1, SW1.1, SW2.1, U1.P$1 (GND), U2.1 (SDO/SA0), U2.2 (SDX), U2.3 (SCX), U2.6 (GND), U2.7 (GND), U3.5 (VSS), U4.2 (GND), U5.5 (GND), U5.9 (HEAT_TAB), U5A1.12 (VSSA), U5A1.18 (VSS), U5A1.31 (VSS), U5A1.47 (VSS), U5A1.63 (VSS), USB_MICRO_CONN1.5 (GND), C18.1
- net CHARGER_STAT1: now reaches U3.3 (STAT1)
- net CHARGER_STAT1: now also U5A1.35 (PB14)
- net at R15.1, R16.2, U5.3 (ADJ): now also C15.1
- no-connect marks 54 -> 49
Other:
- moved on the sheet: C14, C5, C6, D2, D3, J2, R1, R15, R16, R17, R8, R9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

Commit message: restarting routing
Connections:
- net +5V: no longer J4.3 (Pin_3)
- net GND: no longer J4.1 (Pin_1), J4.4 (Pin_4)
- net TEST_GPIO2: now reaches U5A1.29 (PB10)
- net TEST_GPIO2: now also J4.4 (Pin_4)
- net TEST_GPIO0: now reaches U5A1.61 (PB8)
- net TEST_GPIO0: now also J4.1 (Pin_1)
- net TEST_GPIO1: now reaches U5A1.62 (PB9)
- net TEST_GPIO1: now also J4.3 (Pin_3)
- no-connect marks 49 -> 46
Changed lines of the file:
@@
 	1    0    0    -1
 $EndComp
-$Comp
-L power:GND #PWR0112
-U 1 1 5F27037F
-P 5250 4850
-F 0 "#PWR0112" H 5250 4600 50  0001 C CNN
-F 1 "GND" H 5250 4700 50  0000 C CNN
-F 2 "" H 5250 4850 50  0001 C CNN
-F 3 "" H 5250 4850 50  0001 C CNN
-	1    5250 4850
-	1    0    0    -1
-$EndComp
-Wire Wire Line
-	5350 4500 5250 4500
-Wire Wire Line
-	5250 4500 5250 4800
-Wire Wire Line
-	5350 4800 5250 4800
-Connection ~ 5250 4800
-Wire Wire Line
-	5250 4800 5250 4850
-$Comp
-L power:+5V #PWR0113
-U 1 1 5F27038A
-P 5050 4850
-F 0 "#PWR0113" H 5050 4700 50  0001 C CNN
-F 1 "+5V" H 5065 5023 50  0000 C CNN
-F 2 "" H 5050 4850 50  0001 C CNN
-F 3 "" H 5050 4850 50  0001 C CNN
-	1    5050 4850
-	-1   0    0    1
-$EndComp
-Wire Wire Line
-	5350 4700 5050 4700
-Wire Wire Line
-	5050 4700 5050 4850
-Text GLabel 5350 4600 0    50   Input ~ 0
-ADDR_LED_BACKUP_PWM
 Text GLabel 10000 1750 2    50   Input ~ 0
 GREEN_LED
@@
 NoConn ~ 10000 3350
 NoConn ~ 10000 3450
-NoConn ~ 10000 3750
-NoConn ~ 10000 3850
-NoConn ~ 10000 4150
 NoConn ~ 8700 4450
 NoConn ~ 8700 4350
@@
 NoConn ~ 2600 1300
 NoConn ~ 1650 1500
-NoConn ~ 10000 3950
 Text GLabel 10000 4350 2    50   Input ~ 0
 CHARGER_STAT1
@@
 Wire Wire Line
 	2600 1700 3350 1700
+Text GLabel 10000 3750 2    50   Input ~ 0
+TEST_GPIO0
+Text GLabel 10000 3850 2    50   Input ~ 0
+TEST_GPIO1
+Text GLabel 10000 3950 2    50   Input ~ 0
+TEST_GPIO2
+Text GLabel 5350 4600 0    50   Input ~ 0
+ADDR_LED_BACKUP_PWM
+NoConn ~ 10000 4150
+Text GLabel 5350 4500 0    50   Input ~ 0
+TEST_GPIO0
+Text GLabel 5350 4700 0    50   Input ~ 0
+TEST_GPIO1
+Text GLabel 5350 4800 0    50   Input ~ 0
+TEST_GPIO2
 $EndSCHEMATC

Commit message: doing well actually
Connections:
- net BT_RX: now also J1.2 (Pin_2); no longer J1.3 (Pin_3)
- net RESET: now also J1.6 (Pin_6); no longer J1.7 (Pin_7)
- net SWDIO: now also J1.7 (Pin_7); no longer J1.6 (Pin_6)
- net TEST_GPIO0: now also J4.3 (Pin_3); no longer J4.1 (Pin_1)
- net TEST_GPIO1: now also J4.1 (Pin_1); no longer J4.3 (Pin_3)
- net USART_2_RX: now also J1.3 (Pin_3); no longer J1.1 (Pin_1)
- net USART_2_TX: now also J1.1 (Pin_1); no longer J1.2 (Pin_2)
Changed lines of the file:
@@
 Text GLabel 10000 1250 2    50   Input ~ 0
 ADDR_LED_BACKUP_PWM
-Text GLabel 4900 2350 0    60   Input ~ 0
+Text GLabel 4900 2450 0    60   Input ~ 0
 SWDIO
 Text GLabel 4900 2250 0    60   Input ~ 0
 SWCLK
-Text GLabel 4900 2450 0    60   Input ~ 0
+Text GLabel 4900 2350 0    60   Input ~ 0
 RESET
 Text GLabel 4900 2550 0    50   Input ~ 0
@@
 Wire Wire Line
 	7900 4550 8450 4550
-Text GLabel 4900 1950 0    60   Input ~ 0
+Text GLabel 4900 1850 0    60   Input ~ 0
 USART_2_TX
-Text GLabel 4900 1850 0    60   Input ~ 0
+Text GLabel 4900 2050 0    60   Input ~ 0
 USART_2_RX
 Connection ~ 8450 4250
@@
 Text GLabel 4900 2150 0    50   Input ~ 0
 BT_TX
-Text GLabel 4900 2050 0    50   Input ~ 0
+Text GLabel 4900 1950 0    50   Input ~ 0
 BT_RX
 Text GLabel 3500 6300 2    50   Input ~ 0
@@
 ADDR_LED_BACKUP_PWM
 NoConn ~ 10000 4150
+Text GLabel 5350 4700 0    50   Input ~ 0
+TEST_GPIO0
 Text GLabel 5350 4500 0    50   Input ~ 0
-TEST_GPIO0
-Text GLabel 5350 4700 0    50   Input ~ 0
 TEST_GPIO1
 Text GLabel 5350 4800 0    50   Input ~ 0

Commit message: gonna add gnd now
Parts:
- added TP1: TestPoint, TestPoint:TestPoint_Pad_D1.0mm, symbol Connector:TestPoint
- U2: footprint Package_LGA:LGA-14_3x2.5mm_P0.5mm_LayoutBorder3x4y -> footprints:LGA-14_3x2.5mm_P0.5mm_LayoutBorder3x4y_modded
Connections:
- net +3V3: now also TP1.1
Changed lines of the file:
@@
 F 0 "U2" H 4950 7300 50  0000 L CNN
 F 1 "LSM6DS3" H 5150 6700 50  0000 L CNN
-F 2 "Package_LGA:LGA-14_3x2.5mm_P0.5mm_LayoutBorder3x4y" H 4850 6000 50  0001 L CNN
+F 2 "footprints:LGA-14_3x2.5mm_P0.5mm_LayoutBorder3x4y_modded" H 4850 6000 50  0001 L CNN
 F 3 "www.st.com/resource/en/datasheet/lsm6ds3.pdf" H 5350 6050 50  0001 C CNN
 	1    5250 6700
@@
 Text GLabel 6500 4350 0    50   Input ~ 0
 BATT_ADC_ENABLE
-Text Notes 7150 5600 0    50   ~ 0
+Text Notes 7200 6500 0    50   ~ 0
 BATTERY: \n- 1100mAH, 40.5mm x 41.5mm x 6.1mm, li-po battery. (3.0V - 4.2V)\nhttps://www.digikey.com/product-detail/en/tinycircuits/ASR00008/1832-1044-ND/8680974
 Wire Wire Line
@@
 Text GLabel 5350 4800 0    50   Input ~ 0
 TEST_GPIO2
+$Comp
+L power:+3V3 #PWR0108
+U 1 1 5F08E176
+P 7350 5500
+F 0 "#PWR0108" H 7350 5350 50  0001 C CNN
+F 1 "+3V3" H 7365 5673 50  0000 C CNN
+F 2 "" H 7350 5500 50  0001 C CNN
+F 3 "" H 7350 5500 50  0001 C CNN
+	1    7350 5500
+	0    1    1    0
+$EndComp
+$Comp
+L Connector:TestPoint TP1
+U 1 1 5F0817CD
+P 7350 5500
+F 0 "TP1" V 7545 5574 50  0000 C CNN
+F 1 "TestPoint" V 7454 5574 50  0000 C CNN
+F 2 "TestPoint:TestPoint_Pad_D1.0mm" H 7550 5500 50  0001 C CNN
+F 3 "~" H 7550 5500 50  0001 C CNN
+	1    7350 5500
+	0    -1   -1   0
+$EndComp
 $EndSCHEMATC

Commit message: hw not lookin bad ngl
Parts:
- added TP2: TestPoint, TestPoint:TestPoint_Pad_D1.0mm, symbol Connector:TestPoint
Connections:
- net GND: now also TP2.1
Changed lines of the file:
@@
+	0    -1   -1   0
+$EndComp
+$Comp
+L Connector:TestPoint TP2
+U 1 1 5F09DB21
+P 7350 5850
+F 0 "TP2" V 7545 5924 50  0000 C CNN
+F 1 "TestPoint" V 7454 5924 50  0000 C CNN
+F 2 "TestPoint:TestPoint_Pad_D1.0mm" H 7550 5850 50  0001 C CNN
+F 3 "~" H 7550 5850 50  0001 C CNN
+	1    7350 5850
+	0    -1   -1   0
+$EndComp
+$Comp
+L power:GND #PWR0112
+U 1 1 5F0B5555
+P 7350 5850
+F 0 "#PWR0112" H 7350 5600 50  0001 C CNN
+F 1 "GND" H 7355 5677 50  0000 C CNN
+F 2 "" H 7350 5850 50  0001 C CNN
+F 3 "" H 7350 5850 50  0001 C CNN
+	1    7350 5850
 	0    -1   -1   0
 $EndComp
